File: KiCAD/Dual encoder controller.kicad_pcb (KiCad board)
At the start: 2 copper layers, 100 x 100 mm, 9 parts, among them J1 8P8C_Shielded, J2 8P8C_Shielded, J4 2.5x5.5 Barrel Jack, SW1 B3J-3300, U1 Itsy_Bitsy_32u4

Commit message: Add encoder bypass and guard vias
Parts:
- added C1: C_Small, Capacitor_THT:C_Rect_L4.0mm_W2.5mm_P2.50mm, F.Cu at (167.2, 89.7)
- added LOGO1: CC license, Custom Footprints:Creative_commons_license, F.Cu at (182.2, 145.2)
- added LOGO3: OSHW Logo, Symbol:OSHW-Logo2_7.3x6mm_SilkScreen, F.Cu at (190.0, 146.8)
- moved LOGO2 0.10 mm to (155.3, 59.8)
Routing:
- net +5V: track 160.9 -> 165.8 mm
- net /A1: track 55.5 -> 56.5 mm
- net GND: vias 280 -> 400
Other:
- board text added: "License: Creative Commons Attribution-ShareAlike 4.0 https://github.com/Llamero/Dual_encoder_controller Designed by: Benjamin E. Smith, Funded by: NIH P30EY003176"
- board text added: "← Second Encoder"
- board text added: "↑ I2C to LED Driver"
- board text removed: "License: Creative Commons Attribution-ShareAlike 4.0 https://github.com/Llamero/Four_Channel_MHz_LED_Driver Designed by: Benjamin E. Smith, Funded by: NIH P30EY003176"

Commit message: Finished working draft
Other:
- board text added: "ItsyBitsy 32u4 5V"
Changed lines of the file:
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@@
   (gr_line (start 215 60) (end 115 140)
     (stroke (width 0.15) (type default)) (layer "User.1"))
+  (gr_text "ItsyBitsy 32u4 5V" (at 175.06 61.67) (layer "F.SilkS")
+    (effects (font (size 1.5 1.5) (thickness 0.2)) (justify left bottom))
+  )
   (gr_text "6-12V DC" (at 149.66 64.12) (layer "F.SilkS")
     (effects (font (size 1.5 1.5) (thickness 0.2)) (justify left bottom))
